File: KiCad_Files/at90usb1286_prototype/at90USB1286_prototype/at90USB1286_prototype.sch (KiCad schematic (older format))
At the start: 45 parts, among them J1 USB_C_Receptacle_USB2.0, J2 Conn_01x09, J3 Conn_01x03, K1 KEYSW, K2 KEYSW, K3 KEYSW, K4 KEYSW, SW1 SW_Push, U1 AT90USB1286-AU, U2 IS31FL3731-QF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

Commit message: Changed matrix I2C, and finished PCB
Parts:
- removed J3: Conn_01x03, Connector_PinHeader_1.27mm:PinHeader_1x03_P1.27mm_Vertical, symbol Connector_Generic:Conn_01x03
- removed U2: IS31FL3731-QF, Package_DFN_QFN:QFN-28-1EP_4x4mm_P0.4mm_EP2.3x2.3mm, symbol Driver_LED:IS31FL3731-QF
- added C14, C15: 4.7u, Capacitor_SMD:C_0805_2012Metric_Pad1.15x1.40mm_HandSolder, symbol Device:C_Small
- added J3: Conn_01x02, Connector_PinHeader_1.27mm:PinHeader_1x02_P1.27mm_Vertical, symbol Connector_Generic:Conn_01x02
- added U2: IS31FL3733-QF, Package_DFN_QFN:QFN-48-1EP_6x6mm_P0.4mm_EP4.2x4.2mm, symbol Driver_LED:IS31FL3733-QF
- C10: value 0.1u -> 4.7u
- C11: value 10u -> 0.1u
- C12: value 10u -> 4.7u
- C9: value 0.22u -> 0.1u
- K1, K2, K3, K4: footprint Button_Switch_Keyboard:SW_Cherry_MX_1.00u_Plate -> MX_Only:MXOnly-1U-Hotswap; symbol keyboard_parts:KEYSW -> at90USB1286_prototype-rescue:KEYSW-keyboard_parts
- LED1: value C1-1 -> 1A; footprint LED_THT:LED_D1.8mm_W3.3mm_H2.4mm -> MX_Only:MXOnly-LEDONLY
- LED2: value C1-2 -> 2A; footprint LED_THT:LED_D1.8mm_W3.3mm_H2.4mm -> MX_Only:MXOnly-LEDONLY
- LED3: value C2-1 -> 1B; footprint LED_THT:LED_D1.8mm_W3.3mm_H2.4mm -> MX_Only:MXOnly-LEDONLY
- LED4: value C2-2 -> 2B; footprint LED_THT:LED_D1.8mm_W3.3mm_H2.4mm -> MX_Only:MXOnly-LEDONLY
Connections:
- net IN is gone; now on net VCC: C9.2
- net GND: now also C10.1, C9.1, R10.2, C14.1, C15.2, U2.12 (PGND), U2.34 (AGND), U2.43 (ADDR1), U2.44 (ADDR2), U2.48 (GND), U2.49 (GND), U2.5 (PGND); no longer C10.2
- net INTB: now also J3.1 (Pin_1), U2.45 (~INTB)
- net SCK: now also U2.42 (SCL)
- net SDA: now also U2.41 (SDA)
- net SDB: now also J3.2 (Pin_2), U2.46 (~SDB)
- net VCC: now also C10.2, C14.2, C15.1, U2.20 (PVCC), U2.29 (PVCC), U2.37 (AVCC), U2.38 (DVCC), U2.39 (VIO); no longer R10.2
- net at R11.1: now also U2.47 (IICRST)
- net at R12.1: now also U2.35 (RSET)
- net CS2: now reaches LED2.2 (A), LED4.2 (A)
- net CS2: now also U2.17 (CS2)
- net CA1 renamed SW1
- net SW1: now also U2.2 (SW1); no longer LED3.2 (A)
- net CA2 renamed SW2
- net SW2: now also U2.3 (SW2); no longer LED1.2 (A)
- new net CS1: LED1.2 (A), LED3.2 (A), U2.16 (CS1)
- no-connect marks 56 -> 65
Other:
- note added: "Decoupling Capacitors?\n"
- moved on the sheet: LED1, LED2, LED3, LED4, R10, R11, R12, R7, R8, R9
